File: PCB_F107_LAN8720/PCB_F107_LAN8720.kicad_pcb (KiCad board)
At the start: 2 copper layers, 79 parts, among them IC1 LAN8720A, J1 RJ45_HR911105A, J2 485, J3 Conn_01x03, J4 USB_B, SW1 RESET, U1 NCP1117ST33T3G, U2 STM32F107RC_Short_Name, U3 ADM3485, U4 CC1101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

Commit message: working schematic
Parts:
- added D3: BZX84-C5V1, Diode_SMD:D_SOT-23_ANK, B.Cu at (69.5, 32.4)
- added J5: ., Connector_Wire:SolderWirePad_1x01_SMD_1x2mm, F.Cu at (73.7, 46.1)
- added J6: ., Connector_Wire:SolderWirePad_1x01_SMD_1x2mm, F.Cu at (71.7, 46.1)
- added J7: Power, belkin:KF350x2, F.Cu at (69.5, 29.0)
- added J8: DBG, Connector_PinHeader_2.54mm:PinHeader_1x08_P2.54mm_Vertical, F.Cu at (89.0, 57.7)
- BT1: footprint Battery:Battery_Panasonic_CR2032-VS1N_Vertical_CircularHoles -> belkin:2032_vertical
- J3: value Conn_01x03 -> .; footprint Connector_PinSocket_2.00mm:PinSocket_1x03_P2.00mm_Vertical_SMD_Pin1Left -> Connector_Wire:SolderWirePad_1x01_SMD_1x2mm
- U4: footprint Package_DFN_QFN:ST_UFQFPN-20_3x3mm_P0.5mm -> belkin:cc1101
- moved BT1 11.5 mm to (55.8, 36.2), turned to 0 degrees
- moved R18 6.16 mm to (79.1, 43.0), turned to 180 degrees
- moved U1 5.52 mm to (80.0, 30.0)
- moved C22 5.51 mm to (85.2, 28.9)
- moved C11 5.48 mm to (86.9, 28.9)
- moved J3 5.36 mm to (75.7, 46.1)
- moved J4 5.35 mm to (84.3, 39.2)
- moved C13 5.28 mm to (86.3, 32.3)
- moved C12 5.23 mm to (86.5, 34.1)
- moved R20 4.61 mm to (79.1, 43.0), turned to 180 degrees
- moved R19 4.45 mm to (79.1, 45.0), turned to 180 degrees
- moved AE1 2.13 mm to (46.3, 45.4), turned to 180 degrees
- moved C2 1.55 mm to (63.5, 46.0)
- moved C23 1.49 mm to (74.6, 49.6), turned to 90 degrees
- moved C16 1.39 mm to (65.3, 58.0)
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Connections:
- net /RFI1 renamed Net-(U4-Pad6)
- net /RFI2 renamed Net-(U4-Pad3)
- R18 pad 2: /USB_DM -> /USB_DP
- R19 pad 2: /USB_DP -> /USB_DM
- U2 pad 26: Net-(U2-Pad26) -> /PB0
- U2 pad 27: /PHY_nRST -> /PB1
- U2 pad 29: Net-(U2-Pad29) -> /PHY_nRST
- U2 pad 35: Net-(U2-Pad35) -> /PB14
- U2 pad 36: Net-(U2-Pad36) -> /PB15
- U2 pad 37: Net-(U2-Pad37) -> /PC6
- U2 pad 38: Net-(U2-Pad38) -> /PC7
- U2 pad 39: Net-(U2-Pad39) -> /PC8
- U2 pad 40: Net-(U2-Pad40) -> /PC9
Routing:
- net VCC: track 134.1 -> 209.5 mm, vias 13 -> 14
- net GND: track 221.7 -> 184.1 mm, vias 10 -> 13
- net /VBUS: track 25.5 -> 57.4 mm
- net /PC9: track 0.00 -> 21.6 mm
- net /PC8: track 0.00 -> 18.8 mm
- net /PC7: track 0.00 -> 15.7 mm
- net /PC6: track 0.00 -> 13.8 mm
- net /PB14: track 0.00 -> 12.2 mm
- net /PB15: track 0.00 -> 11.6 mm
- net Net-(BT1-Pad1): track 82.9 -> 74.4 mm
- net /USB_DP: track 4.31 -> 12.3 mm
- net /JTMS/SWDIO: track 16.1 -> 8.35 mm
- net /PB1: track 0.00 -> 7.42 mm
- net /PB0: track 0.00 -> 5.62 mm
- net /USB_DM: track 5.74 -> 9.77 mm
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
Commit message: leds
Parts:
- added D4: LED, LED_SMD:LED_0603_1608Metric_Pad1.05x0.95mm_HandSolder, F.Cu at (47.4, 56.3)
- added D5: LED, LED_SMD:LED_0603_1608Metric_Pad1.05x0.95mm_HandSolder, F.Cu at (47.4, 58.2)
- added D6: LED, LED_SMD:LED_0603_1608Metric_Pad1.05x0.95mm_HandSolder, F.Cu at (47.4, 60.2)
- added R12: 100, Resistor_SMD:R_0805_2012Metric_Pad1.15x1.40mm_HandSolder, F.Cu at (50.9, 56.3)
- added R13: 100, Resistor_SMD:R_0805_2012Metric_Pad1.15x1.40mm_HandSolder, F.Cu at (50.9, 58.2)
- added R21: 100, Resistor_SMD:R_0805_2012Metric_Pad1.15x1.40mm_HandSolder, F.Cu at (50.9, 60.2)
- moved BT1 6.68 mm to (55.0, 29.6)
- moved J6 6.17 mm to (68.6, 40.8)
- moved J5 6.06 mm to (70.8, 40.8)
- moved J3 6.04 mm to (72.9, 40.7)
- moved C3 3.98 mm to (83.4, 87.4)
- moved AE1 3.73 mm to (46.3, 41.7)
- moved C15 3.73 mm to (69.1, 48.8)
- moved C16 3.73 mm to (65.3, 54.2)
- moved C2 3.73 mm to (63.5, 42.3)
- moved C25 3.73 mm to (58.0, 37.6)
- moved C26 3.73 mm to (58.0, 42.7)
- moved C27 3.73 mm to (69.1, 47.3)
- moved C28 3.73 mm to (56.1, 48.9)
- moved C29 3.73 mm to (56.1, 45.5)
- moved C30 3.73 mm to (53.7, 53.2)
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Connections:
- D1 pad : (no net) -> GND
- D2 pad : (no net) -> GND
- D3 pad : GND -> (no net)
- U2 pad 54: Net-(U2-Pad54) -> /led1
- U2 pad 55: Net-(U2-Pad55) -> /led2
- U2 pad 56: Net-(U2-Pad56) -> /led3
Routing:
- net GND: track 184.1 -> 158.4 mm, vias 13 -> 14
- net /led1: track 0.00 -> 23.4 mm
- net /led2: track 0.00 -> 22.3 mm
- net /led3: track 0.00 -> 21.6 mm
- net /JTCK/SWCLK: track 11.1 -> 19.4 mm
- net /JTMS/SWDIO: track 8.35 -> 16.4 mm
- net Net-(BT1-Pad1): track 74.4 -> 80.2 mm
- net /NSS: track 18.2 -> 23.5 mm
- net /MISO: track 15.5 -> 20.4 mm
- net VCC: track 209.5 -> 213.1 mm
- net /PHY_nINT: track 30.2 -> 27.0 mm
- net /MDC: track 30.1 -> 26.9 mm
- net /MOSI: track 10.2 -> 13.4 mm
- net /CLK_50M: track 88.4 -> 85.5 mm
- net /SCK: track 9.63 -> 12.4 mm
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
Commit message: libraries
Parts:
- moved BT1 1.98 mm to (55.0, 31.5)
- moved R14 1.02 mm to (62.4, 77.8), turned to 180 degrees
- moved C16 0.47 mm to (65.0, 54.6)
- moved R10 0.24 mm to (63.3, 54.4)
Connections:
- U2 pad 50: /NSS -> Net-(U2-Pad50)
- U2 pad 61: Net-(U2-Pad61) -> /NSS
Routing:
- net VCC: track 213.1 -> 271.4 mm
- net /NSS: track 23.5 -> 32.2 mm, vias 0 -> 2
- net GND: track 158.4 -> 153.6 mm
- net /UART_RX: track 18.1 -> 22.2 mm
- net /MISO: track 20.4 -> 18.0 mm
- net /VBUS: track 57.4 -> 58.8 mm
- net /PC8: track 18.8 -> 20.1 mm
- net Net-(BT1-Pad1): track 80.2 -> 79.1 mm
- net /485RST: track 23.0 -> 24.1 mm
- net /PC9: track 21.6 -> 22.7 mm
- net /PC7: track 15.7 -> 16.7 mm
